Commit message: change repo name

File: fpga_bot_description/urdf/FPGA_bot.urdf (robot description, URDF)
Before this commit: robot FPGA_bot, 11 links, 10 joints
Links:
- link 2nd_motor_arm90deg: geometry collision mesh filename=package://moveit_bot_fpga_bot_description/meshes/2nd_motor_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 scale=0.001 0.001 0.001; visual mesh filename=package://moveit_bot_fpga_bot_description/meshes/2nd_motor_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 scale=0.001 0.001 0.001
- link AX-12A-02: geometry collision mesh filename=package://moveit_bot_fpga_bot_description/meshes/AX-12A-02.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 scale=0.001 0.001 0.001; visual mesh filename=package://moveit_bot_fpga_bot_description/meshes/AX-12A-02.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 scale=0.001 0.001 0.001
- link AX-12A-021: geometry collision mesh filename=package://moveit_bot_fpga_bot_description/meshes/AX-12A-021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 scale=0.001 0.001 0.001; visual mesh filename=package://moveit_bot_fpga_bot_description/meshes/AX-12A-021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 scale=0.001 0.001 0.001
- link AX-12A-022: geometry collision mesh filename=package://moveit_bot_fpga_bot_description/meshes/AX-12A-022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 scale=0.001 0.001 0.001; visual mesh filename=package://moveit_bot_fpga_bot_description/meshes/AX-12A-022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 scale=0.001 0.001 0.001
- link AX-12A-04: geometry collision mesh filename=package://moveit_bot_fpga_bot_description/meshes/AX-12A-04.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 scale=0.001 0.001 0.001; visual mesh filename=package://moveit_bot_fpga_bot_description/meshes/AX-12A-04.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 scale=0.001 0.001 0.001
- link AX-12A-041: geometry collision mesh filename=package://moveit_bot_fpga_bot_description/meshes/AX-12A-041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 scale=0.001 0.001 0.001; visual mesh filename=package://moveit_bot_fpga_bot_description/meshes/AX-12A-041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 scale=0.001 0.001 0.001
- link AX-12A-042: geometry collision mesh filename=package://moveit_bot_fpga_bot_description/meshes/AX-12A-042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 scale=0.001 0.001 0.001; visual mesh filename=package://moveit_bot_fpga_bot_description/meshes/AX-12A-042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 scale=0.001 0.001 0.001
- link Motor_holder_plate: geometry collision mesh filename=package://moveit_bot_fpga_bot_description/meshes/Motor_hold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 scale=0.001 0.001 0.001; visual mesh filename=package://moveit_bot_fpga_bot_description/meshes/Motor_hold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 scale=0.001 0.001 0.001
- link new_2nd_arm_bothsamedirection-v1: geometry collision mesh filename=package://moveit_bot_fpga_bot_description/meshes/new_2nd_ar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 scale=0.001 0.001 0.001; visual mesh filename=package://moveit_bot_fpga_bot_description/meshes/new_2nd_ar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 scale=0.001 0.001 0.001
- link pencil_holder_v2: geometry collision mesh filename=package://moveit_bot_fpga_bot_description/meshes/pencil_hol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 scale=0.001 0.001 0.001; visual mesh filename=package://moveit_bot_fpga_bot_description/meshes/pencil_hol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 scale=0.001 0.001 0.001
- link plate: geometry collision mesh filename=package://moveit_bot_fpga_bot_description/meshes/plate.stl scale=0.001 0.001 0.001; visual mesh filename=package://moveit_bot_fpga_bot_description/meshes/plate.stl scale=0.001 0.001 0.001

File: fpga_bot_moveit_config/config/FPGA_bot.urdf.xacro (robot description, xacro)
@@ -3,5 +3,5 @@
     <xacro:arg name="initial_positions_file" default="initial_positions.yaml" />
     <!-- Import FPGA_bot urdf file -->
-    <xacro:include filename="$(find fpga_bot_fpga_bot_description)/urdf/FPGA_bot.urdf" />
+    <xacro:include filename="$(find moveit_bot_fpga_bot_description)/urdf/FPGA_bot.urdf" />
     <!-- Import control_xacro -->
     <xacro:include filename="FPGA_bot.ros2_control.xacro" />
