Commit message: one joint working

File: bias_bot_description/urdf/BIAS_bot.urdf (robot description, URDF)
Before this commit: robot URDF_assembly, 15 links, 14 joints
Links:
- removed link Lever_connector-v1
- removed link Lever_connector_2-v1
- removed link XM430-W350-R_body
- removed link XM430-W350-R_body1
- removed link XM430-W350-R_idler
- removed link XM430-W350-R_idler1
- removed link arm_end
- removed link cap
- removed link cap1
- removed link cap_2
- removed link cap_21
- removed link mid_arm
- removed link servo_arm
- removed link servo_arm1
- added link arm, mass 0.5711036137259029; collision mesh filename=package://moveit_bot_bias_bot_description/meshes/arm.stl scale=0.001 0.001 0.001; visual mesh filename=package://moveit_bot_bias_bot_description/meshes/arm.stl scale=0.001 0.001 0.001
- added link joint, mass 0.031171001796121915; collision mesh filename=package://moveit_bot_bias_bot_description/meshes/joint.stl scale=0.001 0.001 0.001; visual mesh filename=package://moveit_bot_bias_bot_description/meshes/joint.stl scale=0.001 0.001 0.001
- link shoulder: mass 0.8217980778720475 -> 1.00209496973953
Joints:
- removed joint XM430-W350-R_body1_Revolute-10
- removed joint XM430-W350-R_body_Revolute-21
- removed joint XM430-W350-R_idler1_Rigid-13
- removed joint XM430-W350-R_idler_Rigid-12
- removed joint cap_2_Revolute-34
- removed joint cap_Revolute-6
- removed joint mid_arm_Rigid-7
- removed joint mid_arm_Rigid-8
- removed joint mid_arm_Rigid-9
- removed joint servo_arm1_Revolute-35
- removed joint servo_arm_Revolute-37
- removed joint shoulder_Rigid-3
- removed joint shoulder_Rigid-4
- removed joint shoulder_Rigid-5
- added joint joint_Revolute-3: type continuous, parent joint, child arm, origin xyz=0.0 -0.024000000000000004 0.0 rpy=0.0 -0.0 0.0, axis -0.0 0.0 -1.0, mimic joint=shoulder_Revolute-1 multiplier=-1.0 offset=0.0
- added joint shoulder_Revolute-1: type continuous, parent shoulder, child joint, origin xyz=0.024 -0.069 0.005 rpy=-3.141592653589793 -1.5707963267948966 0, axis 0.0 0.0 1.0

File: bias_bot_moveit_config/config/new_urdf_assembly.ros2_control.xacro (robot description, xacro)
@@ -1,5 +1,5 @@
 <?xml version="1.0"?>
 <robot xmlns:xacro="http://www.ros.org/wiki/xacro">
-    <xacro:macro name="URDF_assembly_ros2_control" params="name initial_positions_file">
+    <xacro:macro name="new_urdf_assembly_ros2_control" params="name initial_positions_file">
         <xacro:property name="initial_positions" value="${xacro.load_yaml(initial_positions_file)['initial_positions']}"/>
         <ros2_control name="${name}" type="system">
@@ -8,15 +8,8 @@
                 <plugin>mock_components/GenericSystem</plugin>
             </hardware>
-            <joint name="cap_Revolute-6">
+            <joint name="shoulder_Revolute-1">
                 <command_interface name="position"/>
                 <state_interface name="position">
-                  <param name="initial_value">${initial_positions['cap_Revolute-6']}</param>
-                </state_interface>
-                <state_interface name="velocity"/>
-            </joint>
-            <joint name="cap_2_Revolute-34">
-                <command_interface name="position"/>
-                <state_interface name="position">
-                  <param name="initial_value">${initial_positions['cap_2_Revolute-34']}</param>
+                  <param name="initial_value">${initial_positions['shoulder_Revolute-1']}</param>
                 </state_interface>
                 <state_interface name="velocity"/>

Commit message: new arm design

File: bias_bot_description/urdf/BIAS_bot.urdf (robot description, URDF)
Before this commit: robot new_urdf_assembly, 3 links, 2 joints
Links:
- removed link arm
- removed link joint
- removed link shoulder
- added link ArmV3_arm_1_2, mass 0.4561701564775116; collision mesh filename=package://moveit_bot_bias_bot_description/meshes/ArmV3_arm_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 scale=0.001 0.001 0.001; visual mesh filename=package://moveit_bot_bias_bot_description/meshes/ArmV3_arm_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 scale=0.001 0.001 0.001
- added link ArmV3_arm_1_2_3, mass 0.5712342497066363; collision mesh filename=package://moveit_bot_bias_bot_description/meshes/ArmV3_arm_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 scale=0.001 0.001 0.001; visual mesh filename=package://moveit_bot_bias_bot_description/meshes/ArmV3_arm_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 scale=0.001 0.001 0.001
- added link ArmV3_arm_1_main, mass 0.8691619110350246; collision mesh filename=package://moveit_bot_bias_bot_description/meshes/ArmV3_arm_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 scale=0.001 0.001 0.001; visual mesh filename=package://moveit_bot_bias_bot_description/meshes/ArmV3_arm_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 scale=0.001 0.001 0.001
- added link ArmV3_arm_1_main_3, mass 1.0536423016393843; collision mesh filename=package://moveit_bot_bias_bot_description/meshes/ArmV3_arm_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 scale=0.001 0.001 0.001; visual mesh filename=package://moveit_bot_bias_bot_description/meshes/ArmV3_arm_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 scale=0.001 0.001 0.001
- added link Joint, mass 0.033587469088615846; collision mesh filename=package://moveit_bot_bias_bot_description/meshes/Joint.stl scale=0.001 0.001 0.001; visual mesh filename=package://moveit_bot_bias_bot_description/meshes/Joint.stl scale=0.001 0.001 0.001
- added link Joint1, mass 0.033587469088615846; collision mesh filename=package://moveit_bot_bias_bot_description/meshes/Joint1.stl scale=0.001 0.001 0.001; visual mesh filename=package://moveit_bot_bias_bot_description/meshes/Joint1.stl scale=0.001 0.001 0.001
- added link Joint3, mass 0.033587469088615846; collision mesh filename=package://moveit_bot_bias_bot_description/meshes/Joint3.stl scale=0.001 0.001 0.001; visual mesh filename=package://moveit_bot_bias_bot_description/meshes/Joint3.stl scale=0.001 0.001 0.001
- added link Pulley, mass 0.08716626706769168; collision mesh filename=package://moveit_bot_bias_bot_description/meshes/Pulley.stl scale=0.001 0.001 0.001; visual mesh filename=package://moveit_bot_bias_bot_description/meshes/Pulley.stl scale=0.001 0.001 0.001
- added link Pulley1, mass 0.08716626706769168; collision mesh filename=package://moveit_bot_bias_bot_description/meshes/Pulley1.stl scale=0.001 0.001 0.001; visual mesh filename=package://moveit_bot_bias_bot_description/meshes/Pulley1.stl scale=0.001 0.001 0.001
- added link Pulley2, mass 0.08716626706769168; collision mesh filename=package://moveit_bot_bias_bot_description/meshes/Pulley2.stl scale=0.001 0.001 0.001; visual mesh filename=package://moveit_bot_bias_bot_description/meshes/Pulley2.stl scale=0.001 0.001 0.001
- added link Servo_dummy, mass 0.35035104472812495; collision mesh filename=package://moveit_bot_bias_bot_description/meshes/Servo_dumm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 scale=0.001 0.001 0.001; visual mesh filename=package://moveit_bot_bias_bot_description/meshes/Servo_dumm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 scale=0.001 0.001 0.001
- added link Servo_dummy2, mass 0.35035104472812495; collision mesh filename=package://moveit_bot_bias_bot_description/meshes/Servo_dumm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 scale=0.001 0.001 0.001; visual mesh filename=package://moveit_bot_bias_bot_description/meshes/Servo_dumm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 scale=0.001 0.001 0.001
- added link Servo_dummy3, mass 0.35035104472812495; collision mesh filename=package://moveit_bot_bias_bot_description/meshes/Servo_dumm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 scale=0.001 0.001 0.001; visual mesh filename=package://moveit_bot_bias_bot_description/meshes/Servo_dumm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 scale=0.001 0.001 0.001
- added link Servo_dummy4, mass 0.35035104472812495; collision mesh filename=package://moveit_bot_bias_bot_description/meshes/Servo_dumm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 scale=0.001 0.001 0.001; visual mesh filename=package://moveit_bot_bias_bot_description/meshes/Servo_dumm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 scale=0.001 0.001 0.001
- added link Shoulder; collision mesh filename=package://moveit_bot_bias_bot_description/meshes/Shoulder.s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 scale=0.001 0.001 0.001; visual mesh filename=package://moveit_bot_bias_bot_description/meshes/Shoulder.s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 scale=0.001 0.001 0.001
- added link Shoulder_joint, mass 0.5711036137259029; collision mesh filename=package://moveit_bot_bias_bot_description/meshes/Shoulder_j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 scale=0.001 0.001 0.001; visual mesh filename=package://moveit_bot_bias_bot_description/meshes/Shoulder_j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 scale=0.001 0.001 0.001
- added link Wire_support_R, mass 0.11933054574035153; collision mesh filename=package://moveit_bot_bias_bot_description/meshes/Wire_suppo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 scale=0.001 0.001 0.001; visual mesh filename=package://moveit_bot_bias_bot_description/meshes/Wire_suppo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 scale=0.001 0.001 0.001
- added link Wire_support_R1, mass 0.11933054574035153; collision mesh filename=package://moveit_bot_bias_bot_description/meshes/Wire_suppo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 scale=0.001 0.001 0.001; visual mesh filename=package://moveit_bot_bias_bot_description/meshes/Wire_suppo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 scale=0.001 0.001 0.001
- added link Wire_support_R2, mass 0.11933054574035153; collision mesh filename=package://moveit_bot_bias_bot_description/meshes/Wire_suppo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 scale=0.001 0.001 0.001; visual mesh filename=package://moveit_bot_bias_bot_description/meshes/Wire_suppo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 scale=0.001 0.001 0.001
- added link end, mass 0.056453498805117096; collision mesh filename=package://moveit_bot_bias_bot_description/meshes/end.stl scale=0.001 0.001 0.001; visual mesh filename=package://moveit_bot_bias_bot_description/meshes/end.stl scale=0.001 0.001 0.001
- added link wrist, mass 0.32553675299285556; collision mesh filename=package://moveit_bot_bias_bot_description/meshes/wrist.stl scale=0.001 0.001 0.001; visual mesh filename=package://moveit_bot_bias_bot_description/meshes/wrist.stl scale=0.001 0.001 0.001
Joints:
- removed joint joint_Revolute-3
- removed joint shoulder_Revolute-1
- added joint ArmV3_arm_1_2_3_Rigid-18: type fixed, parent ArmV3_arm_1_2_3, child wrist, origin xyz=-0.013500000000000002 0.024000000000000004 -0.06350000000000001 rpy=-3.141592653589793 -1.5707963267948966 0
- added joint ArmV3_arm_1_2_Rigid-12: type fixed, parent ArmV3_arm_1_2, child ArmV3_arm_1_main_3, origin xyz=-0.013500000000000002 0.024000000000000004 -0.0635 rpy=-3.141592653589793 -1.5707963267948966 0
- added joint ArmV3_arm_1_main_3_Revolute-16: type continuous, parent ArmV3_arm_1_main_3, child Joint3, origin xyz=-0.06457456 0.024000000000000004 -0.0022727100000000003 rpy=-1.5707963267948966 -0.0 4.3790577010150533e-47, axis 4.3790577010150533e-47 -9.860761315262648e-32 1.0
- added joint ArmV3_arm_1_main_3_Rigid-13: type fixed, parent ArmV3_arm_1_main_3, child Servo_dummy2, origin xyz=0.021967239999999996 0.00584257 0.06055392 rpy=0.0 0.6981317007977311 -3.141592653589793
- added joint ArmV3_arm_1_main_Revolute-10: type continuous, parent ArmV3_arm_1_main, child Joint1, origin xyz=-0.0605 -0.0025 0.044000000000000004 rpy=0.0 -7.87425696643208e-47 0.0, axis 7.810989099284927e-47 0.0 1.0
- added joint ArmV3_arm_1_main_Rigid-7: type fixed, parent ArmV3_arm_1_main, child Servo_dummy3, origin xyz=0.046171090000000005 0.005 0.025763820000000003 rpy=1.5707963267948966 -7.87425696643208e-47 0.0
- added joint Joint1_Revolute-11: type continuous, parent Joint1, child ArmV3_arm_1_2, origin xyz=-0.024000000000000004 0.0 0.0 rpy=-1.5707963267948966 -0.0 -1.5707963267948966, axis 0.0 1.0 0.0, mimic joint=ArmV3_arm_1_main_Revolute-10 multiplier=-1.0 offset=0.0
- added joint Joint3_Revolute-17: type continuous, parent Joint3, child ArmV3_arm_1_2_3, origin xyz=-0.023999999999999987 0.0 0.0 rpy=-1.5707963267948966 1.4791141972893971e-31 -1.5707963267948966, axis 4.930380657631324e-32 1.0 0.0, mimic joint=ArmV3_arm_1_main_3_Revolute-16 multiplier=-1.0 offset=0.0
- added joint Joint_Revolute-2: type continuous, parent Joint, child Shoulder_joint, origin xyz=0.0 -0.024000000000000004 0.0 rpy=0.0 -0.0 0.0, axis 0.0 0.0 -1.0, mimic joint=Shoulder_Revolute-1 multiplier=-1.0 offset=0.0
- added joint Servo_dummy2_Rigid-14: type fixed, parent Servo_dummy2, child Wire_support_R2, origin xyz=-0.024000000659561885 0.0 0.02850000041077772 rpy=-5.551115123125783e-17 -0.8726646259971654 3.141592653589793
- added joint Servo_dummy2_Rigid-15: type fixed, parent Servo_dummy2, child Pulley2, origin xyz=0.012000003769883812 -0.012999999999999998 0.014250000554834177 rpy=-4.6579386524374596e-17 0.6981317007977311 3.141592653589793
- added joint Servo_dummy3_Rigid-8: type fixed, parent Servo_dummy3, child Wire_support_R1, origin xyz=0.0 0.0 0.0285 rpy=3.0814879110194994e-33 -1.5707963267948966 0
- added joint Servo_dummy3_Rigid-9: type fixed, parent Servo_dummy3, child Pulley1, origin xyz=-0.012000000000000002 0.012999999999999998 0.01425 rpy=8.602605125365621e-33 1.9721522630525295e-31 3.0814879110194994e-33
- added joint Servo_dummy4_Revolute-20: type continuous, parent Servo_dummy4, child end, origin xyz=-0.013000000000000043 0.004 0.014250000000000002 rpy=3.141592653589793 -0.0 -8.776337004300883e-32, axis -1.0 -0.0 0.0
- added joint Servo_dummy_Rigid-4: type fixed, parent Servo_dummy, child Pulley, origin xyz=0.012999999999999998 0.01200000000000001 0.01425 rpy=-1.9721522630525295e-31 -0.0 -2.088097429759528e-53
- added joint Servo_dummy_Rigid-5: type fixed, parent Servo_dummy, child Wire_support_R, origin xyz=0.0 0.0 0.0285 rpy=-2.088097429759528e-53 -1.5707963267948966 0
- added joint Shoulder_Revolute-1: type continuous, parent Shoulder, child Joint, origin xyz=0.024 -0.069 0.005 rpy=-3.141592653589793 -1.5707963267948966 0, axis 0.0 0.0 1.0
- added joint Shoulder_Rigid-3: type fixed, parent Shoulder, child Servo_dummy, origin xyz=0.006 -0.114 0.0 rpy=0.0 -0.0 0.0
- added joint Shoulder_joint_Rigid-6: type fixed, parent Shoulder_joint, child ArmV3_arm_1_main, origin xyz=0.0 -0.045 -0.016 rpy=1.5707963267948966 -1.5707963267948966 0
- added joint wrist_Rigid-19: type fixed, parent wrist, child Servo_dummy4, origin xyz=-0.038920109999999966 -0.02773716 -0.003999999999999999 rpy=-3.141592653589793 -4.930380657631324e-32 2.2625809587726806e-32

Commit message: add crystal

File: bias_bot_description/urdf/BIAS_bot.urdf (robot description, URDF)
Before this commit: robot BIAS_bot, 21 links, 20 joints
Links:
- removed link end
- added link Crystal, mass 0.08850536048231127; collision mesh filename=package://moveit_bot_bias_bot_description/meshes/Crystal.stl scale=0.001 0.001 0.001; visual mesh filename=package://moveit_bot_bias_bot_description/meshes/Crystal.stl scale=0.001 0.001 0.001
- added link crystal_holder, mass 0.1047728661895372; collision mesh filename=package://moveit_bot_bias_bot_description/meshes/crystal_ho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 scale=0.001 0.001 0.001; visual mesh filename=package://moveit_bot_bias_bot_description/meshes/crystal_ho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 scale=0.001 0.001 0.001
Joints:
- added joint crystal_holder_Rigid-21: type fixed, parent crystal_holder, child Crystal, origin xyz=-0.006000009999999989 -0.00024999999999999914 -0.038051009999999996 rpy=-3.141592653589793 4.867941253436161e-62 -1.2338329337763984e-31
- joint Servo_dummy4_Revolute-20: child end -> crystal_holder
